File: auto-water.kicad_sch (KiCad schematic)
At the start: 6 parts, among them J1 ESP32_GPIO4, J2 LOAD, K1 SRD-05VDC-SL-C, Q1 2N2222A

Commit message: add float and water endpoints for testing
Parts:
- J1: value ESP32_GPIO4 -> ESP32_GPIO26
Other:
- note added: "ESP32 GPIO26 drives transistor base through 1kΩ current-limiting resistor"
- note removed: "ESP32 GPIO4 drives transistor base through 1kΩ current-limiting resistor"
Changed lines of the file:
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@@
 		)
 	)
-	(text "ESP32 GPIO4 drives transistor base\nthrough 1kΩ current-limiting resistor"
+  (text "ESP32 GPIO26 drives transistor base\nthrough 1kΩ current-limiting resistor"
 		(exclude_from_sim no)
 		(at 93.98 101.6 0)
@@
 			)
 		)
-		(property "Value" "ESP32_GPIO4"
+		(property "Value" "ESP32_GPIO26"
 			(at 101.6 93.98 0)
 			(show_name no)
